File: hardware/avr-watch.brd (EAGLE design)
At the start: 31.5 x 38.1 mm, 43 parts, among them IC1 MEGA48/88/168-AU, Q5 32k, U1 MAX1555

Commit message: hardware: cosmetic changes, add pdf
Parts:
- Q5: value 32k -> 12MHz
Changed lines of the file:
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@@
 <element name="S1" library="sparkfun" package="TACTILE_SWITCH_SMD" value="SWITCH-MOMENTARY-2SMD" x="28.8544" y="16.1036" rot="R90"/>
 <element name="S2" library="sparkfun" package="TACTILE_SWITCH_SMD" value="SWITCH-MOMENTARY-2SMD" x="28.8544" y="9.1948" rot="R270"/>
-<element name="Q5" library="crystal" package="CTS406" value="32k" x="22.5429" y="9.1528" rot="R45"/>
+<element name="Q5" library="crystal" package="CTS406" value="12MHz" x="22.5429" y="9.1528" rot="R45"/>
 <element name="C1" library="rcl" package="C0805" value="22p" x="21.1328" y="7.9756" rot="MR0"/>
 <element name="R1" library="rcl" package="R0603" value="68" x="7.3152" y="13.6652" rot="MR180"/>
